File: hochzeits-pcb/hochzeits-pcb.kicad_sch (KiCad schematic)
At the start: 5 parts, among them SW1 SW_DIP_x01

Commit message: feat: layout done
Other:
- note added: "Hochzeit Sandra & Markus 14.08.2026"
Changed lines of the file:
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@@
 		(title "Hochzeit Sandra+Markus ")
+	)
+	(text "Hochzeit\nSandra & Markus\n14.08.2026"
+		(exclude_from_sim no)
+		(at 131.826 105.41 0)
+		(effects
+			(font
+				(size 1.27 1.27)
+			)
+		)
 	)
 	(junction
@@
 		(color 0 0 0 0)
 	)
+	(bus_entry
+		(at 120.65 91.44)
+		(size 2.54 2.54)
+		(stroke
+			(width 0)
+			(type default)
+		)
+	)
 	(wire
